File: mini-lab-diy.kicad_sch (KiCad schematic)
At the start: 68 parts, among them J1 Conn_01x20, J2 Conn_01x20, M1 Motor_Servo, SW17 SW_Push_Dual, SW18 SW_Push_Dual, SW19 SW_Push_Dual, SW20 SW_Push_Dual, U3 FRANZININHO_WIFI_PINOUT

Commit message: retirada dos gnd do led rgb e do motor, e aumento no espaçamento dos dados da silk
Parts:
- removed Enable0, Enable1: Conn_01x02, Connector_PinHeader_2.54mm:PinHeader_1x02_P2.54mm_Vertical, symbol Connector_Generic:Conn_01x02
- POT1: footprint Potentiometer_THT:Potentiometer_Alps_RK09Y11_Single_Horizontal -> Potentiometer_THT:Potentiometer_Bourns_PTV09A-1_Single_Vertical
Connections:
- net GND: now also LED5.4 (A), M1.3 (-)
Other:
- moved on the sheet: EnableL4, EnableL5, EnableL6, LED5, R10, R11, R9
